File: pcb/slimy.kicad_pcb (KiCad board)
At the start: 2 copper layers, 91.4 x 96.5 mm, 3 parts, among them U1 Teensy3.2, U2 PIM447, U3 ST7789_SPI

Commit message: WIP keyboard pcb design
Parts:
- added D1: D, my_lib:D_SOD123_axial, F.Cu at (-310.5, 46.0)
- added D10: D, my_lib:D_SOD123_axial, F.Cu at (-83.2, 46.0)
- added D11: D, my_lib:D_SOD123_axial, F.Cu at (-64.1, 46.0)
- added D12: D, my_lib:D_SOD123_axial, F.Cu at (-45.1, 46.0)
- added D13: D, my_lib:D_SOD123_axial, F.Cu at (-310.5, 65.0)
- added D14: D, my_lib:D_SOD123_axial, F.Cu at (-291.5, 65.0)
- added D15: D, my_lib:D_SOD123_axial, F.Cu at (-272.4, 65.0)
- added D16: D, my_lib:D_SOD123_axial, F.Cu at (-253.4, 65.0)
- added D17: D, my_lib:D_SOD123_axial, F.Cu at (-234.3, 65.0)
- added D18: D, my_lib:D_SOD123_axial, F.Cu at (-215.3, 65.0)
- added D19: D, my_lib:D_SOD123_axial, F.Cu at (-140.3, 65.0)
- added D2: D, my_lib:D_SOD123_axial, F.Cu at (-291.5, 46.0)
- added D20: D, my_lib:D_SOD123_axial, F.Cu at (-121.3, 65.0)
- added D21: D, my_lib:D_SOD123_axial, F.Cu at (-102.2, 65.0)
- added D22: D, my_lib:D_SOD123_axial, F.Cu at (-83.2, 65.0)
- added D23: D, my_lib:D_SOD123_axial, F.Cu at (-64.1, 65.0)
- added D24: D, my_lib:D_SOD123_axial, F.Cu at (-45.1, 65.0)
- added D25: D, my_lib:D_SOD123_axial, F.Cu at (-310.5, 84.1)
- added D26: D, my_lib:D_SOD123_axial, F.Cu at (-291.5, 84.1)
- added D27: D, my_lib:D_SOD123_axial, F.Cu at (-272.4, 84.1)
- added D28: D, my_lib:D_SOD123_axial, F.Cu at (-253.4, 84.1)
- added D29: D, my_lib:D_SOD123_axial, F.Cu at (-234.3, 84.1)
- added D3: D, my_lib:D_SOD123_axial, F.Cu at (-272.4, 46.0)
- added D30: D, my_lib:D_SOD123_axial, F.Cu at (-215.3, 84.1)
- added D31: D, my_lib:D_SOD123_axial, F.Cu at (-140.3, 84.1)
- added D32: D, my_lib:D_SOD123_axial, F.Cu at (-121.3, 84.1)
- added D33: D, my_lib:D_SOD123_axial, F.Cu at (-102.2, 84.1)
- added D34: D, my_lib:D_SOD123_axial, F.Cu at (-83.2, 84.1)
- added D35: D, my_lib:D_SOD123_axial, F.Cu at (-64.1, 84.1)
- added D36: D, my_lib:D_SOD123_axial, F.Cu at (-45.1, 84.1)
- added D37: D, my_lib:D_SOD123_axial, F.Cu at (-310.5, 103.1)
- added D38: D, my_lib:D_SOD123_axial, F.Cu at (-291.5, 103.1)
- added D39: D, my_lib:D_SOD123_axial, F.Cu at (-272.4, 103.1)
- added D4: D, my_lib:D_SOD123_axial, F.Cu at (-253.4, 46.0)
- added D40: D, my_lib:D_SOD123_axial, F.Cu at (-253.4, 103.1)
- added D41: D, my_lib:D_SOD123_axial, F.Cu at (-234.3, 103.1)
- added D42: D, my_lib:D_SOD123_axial, F.Cu at (-215.3, 103.1)
- added D43: D, my_lib:D_SOD123_axial, F.Cu at (-140.3, 103.1)
- added D44: D, my_lib:D_SOD123_axial, F.Cu at (-121.3, 103.1)
- added D45: D, my_lib:D_SOD123_axial, F.Cu at (-102.2, 103.1)
- added D46: D, my_lib:D_SOD123_axial, F.Cu at (-83.2, 103.1)
- added D47: D, my_lib:D_SOD123_axial, F.Cu at (-64.1, 103.1)
- added D48: D, my_lib:D_SOD123_axial, F.Cu at (-45.1, 103.1)
- added D49: D, my_lib:D_SOD123_axial, F.Cu at (-215.3, 122.2)
- added D5: D, my_lib:D_SOD123_axial, F.Cu at (-234.3, 46.0)
- added D50: D, my_lib:D_SOD123_axial, F.Cu at (-196.2, 122.2)
- added D51: D, my_lib:D_SOD123_axial, F.Cu at (-196.2, 103.1)
- added D52: D, my_lib:D_SOD123_axial, F.Cu at (-159.4, 103.1)
- added D53: D, my_lib:D_SOD123_axial, F.Cu at (-159.4, 122.2)
- added D54: D, my_lib:D_SOD123_axial, F.Cu at (-140.3, 122.2)
- added D6: D, my_lib:D_SOD123_axial, F.Cu at (-215.3, 46.0)
- added D7: D, my_lib:D_SOD123_axial, F.Cu at (-140.3, 46.0)
- added D8: D, my_lib:D_SOD123_axial, F.Cu at (-121.3, 46.0)
- added D9: D, my_lib:D_SOD123_axial, F.Cu at (-102.2, 46.0)
- added K1: KEYSW, my_lib:MX-1U-Hotswap-Antishear, F.Cu at (-310.5, 54.6)
- added K10: KEYSW, my_lib:MX-1U-Hotswap-Antishear, F.Cu at (-83.2, 54.6)
- added K11: KEYSW, my_lib:MX-1U-Hotswap-Antishear, F.Cu at (-64.1, 54.6)
- added K12: KEYSW, my_lib:MX-1U-Hotswap-Antishear, F.Cu at (-45.1, 54.6)
- added K13: KEYSW, my_lib:MX-1U-Hotswap-Antishear, F.Cu at (-310.5, 73.7)
- added K14: KEYSW, my_lib:MX-1U-Hotswap-Antishear, F.Cu at (-291.5, 73.7)
- added K15: KEYSW, my_lib:MX-1U-Hotswap-Antishear, F.Cu at (-272.4, 73.7)
- added K16: KEYSW, my_lib:MX-1U-Hotswap-Antishear, F.Cu at (-253.4, 73.7)
- added K17: KEYSW, my_lib:MX-1U-Hotswap-Antishear, F.Cu at (-234.3, 73.7)
- added K18: KEYSW, my_lib:MX-1U-Hotswap-Antishear, F.Cu at (-215.3, 73.7)
- added K19: KEYSW, my_lib:MX-1U-Hotswap-Antishear, F.Cu at (-140.3, 73.7)
- added K2: KEYSW, my_lib:MX-1U-Hotswap-Antishear, F.Cu at (-291.5, 54.6)
- added K20: KEYSW, my_lib:MX-1U-Hotswap-Antishear, F.Cu at (-121.3, 73.7)
- added K21: KEYSW, my_lib:MX-1U-Hotswap-Antishear, F.Cu at (-102.2, 73.7)
- added K22: KEYSW, my_lib:MX-1U-Hotswap-Antishear, F.Cu at (-83.2, 73.7)
- added K23: KEYSW, my_lib:MX-1U-Hotswap-Antishear, F.Cu at (-64.1, 73.7)
- added K24: KEYSW, my_lib:MX-1U-Hotswap-Antishear, F.Cu at (-45.1, 73.7)
- added K25: KEYSW, my_lib:MX-1U-Hotswap-Antishear, F.Cu at (-310.5, 92.7)
- added K26: KEYSW, my_lib:MX-1U-Hotswap-Antishear, F.Cu at (-291.5, 92.7)
- added K27: KEYSW, my_lib:MX-1U-Hotswap-Antishear, F.Cu at (-272.4, 92.7)
- added K28: KEYSW, my_lib:MX-1U-Hotswap-Antishear, F.Cu at (-253.4, 92.7)
- added K29: KEYSW, my_lib:MX-1U-Hotswap-Antishear, F.Cu at (-234.3, 92.7)
- added K3: KEYSW, my_lib:MX-1U-Hotswap-Antishear, F.Cu at (-272.4, 54.6)
- added K30: KEYSW, my_lib:MX-1U-Hotswap-Antishear, F.Cu at (-215.3, 92.7)
- added K31: KEYSW, my_lib:MX-1U-Hotswap-Antishear, F.Cu at (-140.3, 92.7)
- added K32: KEYSW, my_lib:MX-1U-Hotswap-Antishear, F.Cu at (-121.3, 92.7)
- added K33: KEYSW, my_lib:MX-1U-Hotswap-Antishear, F.Cu at (-102.2, 92.7)
- added K34: KEYSW, my_lib:MX-1U-Hotswap-Antishear, F.Cu at (-83.2, 92.7)
- added K35: KEYSW, my_lib:MX-1U-Hotswap-Antishear, F.Cu at (-64.1, 92.7)
- added K36: KEYSW, my_lib:MX-1U-Hotswap-Antishear, F.Cu at (-45.1, 92.7)
- added K37: KEYSW, my_lib:MX-1U-Hotswap-Antishear, F.Cu at (-310.5, 111.8)
- added K38: KEYSW, my_lib:MX-1U-Hotswap-Antishear, F.Cu at (-291.5, 111.8)
- added K39: KEYSW, my_lib:MX-1U-Hotswap-Antishear, F.Cu at (-272.4, 111.8)
- added K4: KEYSW, my_lib:MX-1U-Hotswap-Antishear, F.Cu at (-253.4, 54.6)
- added K40: KEYSW, my_lib:MX-1U-Hotswap-Antishear, F.Cu at (-253.4, 111.8)
- added K41: KEYSW, my_lib:MX-1U-Hotswap-Antishear, F.Cu at (-234.3, 111.8)
- added K42: KEYSW, my_lib:MX-1U-Hotswap-Antishear, F.Cu at (-215.3, 111.8)
- added K43: KEYSW, my_lib:MX-1U-Hotswap-Antishear, F.Cu at (-140.3, 111.8)
- added K44: KEYSW, my_lib:MX-1U-Hotswap-Antishear, F.Cu at (-121.3, 111.8)
- added K45: KEYSW, my_lib:MX-1U-Hotswap-Antishear, F.Cu at (-102.2, 111.8)
- added K46: KEYSW, my_lib:MX-1U-Hotswap-Antishear, F.Cu at (-83.2, 111.8)
- added K47: KEYSW, my_lib:MX-1U-Hotswap-Antishear, F.Cu at (-64.1, 111.8)
- added K48: KEYSW, my_lib:MX-1U-Hotswap-Antishear, F.Cu at (-45.1, 111.8)
- added K49: KEYSW, my_lib:MX-1U-Hotswap-Antishear, F.Cu at (-215.3, 130.8)
- added K5: KEYSW, my_lib:MX-1U-Hotswap-Antishear, F.Cu at (-234.3, 54.6)
- added K50: KEYSW, my_lib:MX-1U-Hotswap-Antishear, F.Cu at (-196.2, 130.8)
- added K51: KEYSW, my_lib:MX-1U-Hotswap-Antishear, F.Cu at (-196.2, 111.8)
- added K52: KEYSW, my_lib:MX-1U-Hotswap-Antishear, F.Cu at (-159.4, 111.8)
- added K53: KEYSW, my_lib:MX-1U-Hotswap-Antishear, F.Cu at (-159.4, 130.8)
- added K54: KEYSW, my_lib:MX-1U-Hotswap-Antishear, F.Cu at (-140.3, 130.8)
- added K6: KEYSW, my_lib:MX-1U-Hotswap-Antishear, F.Cu at (-215.3, 54.6)
- added K7: KEYSW, my_lib:MX-1U-Hotswap-Antishear, F.Cu at (-140.3, 54.6)
- added K8: KEYSW, my_lib:MX-1U-Hotswap-Antishear, F.Cu at (-121.3, 54.6)
- added K9: KEYSW, my_lib:MX-1U-Hotswap-Antishear, F.Cu at (-102.2, 54.6)
- U1: value Teensy3.2 -> PIM447; footprint teensy:Teensy30_31_32_All_Pins -> my_lib:PIM447
- U2: renamed from U3; value ST7789_SPI -> Teensy3.2; footprint my_lib:ST7789_1.3_240x240 -> teensy:Teensy30_31_32_All_Pins
- U3: renamed from U2; value PIM447 -> ST7789_SPI; footprint my_lib:PIM447 -> my_lib:ST7789_1.3_240x240
- moved U1 203.7 mm to (183.0, 268.9), turned to 0 degrees
- moved U3 116.0 mm to (183.1, 217.3), turned to 0 degrees
- moved U2 84.2 mm to (182.2, 180.3), turned to -90 degrees
Connections:
- U1 pad 1: GND -> VCC
- U1 pad 2: unconnected-(U1-Pad2) -> SDA
- U1 pad 3: unconnected-(U1-Pad3) -> SCL
- U1 pad 5: unconnected-(U1-Pad5) -> GND
- U2 pad 1: VCC -> GND
- U2 pad 10: unconnected-(U3-Pad10) -> Col5
- U2 pad 11: unconnected-(U3-Pad11) -> LCD LITE
- U2 pad 2: unconnected-(U3-Pad2) -> Row4
- U2 pad 3: GND -> Row3
- U2 pad 4: SCK -> Row2
- U2 pad 5: MISO -> Row1
- U2 pad 6: MOSI -> Col1
- U2 pad 7: LCD CS -> Col2
- U2 pad 8: LCD RST -> Col3
- U2 pad 9: LCD DC -> Col4
- U3 pad 2: SDA -> unconnected-(U3-Pad2)
- U3 pad 3: SCL -> GND
- U3 pad 4: unconnected-(U2-Pad4) -> Row5
- U3 pad 5: GND -> unconnected-(U3-Pad5)
Routing:
- net Row1: track 0.00 -> 213.9 mm
- net Row4: track 0.00 -> 213.9 mm
- net Row2: track 0.00 -> 213.9 mm
- net Row3: track 0.00 -> 213.9 mm
- net Col9: track 0.00 -> 102.0 mm
- net VCC: track 100.7 -> 0.00 mm
- net Col8: track 0.00 -> 100.1 mm
- net Row5: track 0.00 -> 90.7 mm
- net Col6: track 0.00 -> 75.5 mm
- net Col7: track 0.00 -> 73.7 mm
- net Col5: track 0.00 -> 52.6 mm
- net Col4: track 0.00 -> 52.6 mm
- net Col3: track 0.00 -> 52.6 mm
- net Col2: track 0.00 -> 52.6 mm
- net Col12: track 0.00 -> 52.6 mm
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- removed copper zone on F.Cu, net GND
Other:
- board size 91.4 x 96.5 mm -> 284.5 x 95.2 mm

Commit message: First iteration design
Parts:
- moved K53 403.7 mm to (241.6, 177.7), turned to 10 degrees
- moved K54 403.0 mm to (260.3, 174.4), turned to 10 degrees
- moved D53 402.2 mm to (240.1, 169.2), turned to -170 degrees
- moved D54 401.5 mm to (258.8, 165.9), turned to -170 degrees
- moved K52 400.4 mm to (238.2, 158.9), turned to 10 degrees
- moved K43 399.8 mm to (257.0, 155.6), turned to 10 degrees
- moved K44 399.1 mm to (275.8, 152.3), turned to 10 degrees
- moved D52 398.9 mm to (236.7, 150.4), turned to -170 degrees
- moved D6 398.7 mm to (180.9, 90.8), turned to 170 degrees
- moved D5 398.6 mm to (162.1, 87.5), turned to 170 degrees
- moved D1 398.6 mm to (87.1, 74.3), turned to 170 degrees
- moved D4 398.5 mm to (143.3, 84.2), turned to 170 degrees
- moved D2 398.5 mm to (105.8, 77.6), turned to 170 degrees
- moved D3 398.5 mm to (124.6, 80.9), turned to 170 degrees
- moved K45 398.5 mm to (294.5, 149.0), turned to 10 degrees
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Other:
- board size 284.5 x 95.2 mm -> 297.2 x 117 mm

Commit message: First iteration design pt2
Parts:
- moved U1 99.4 mm to (216.0, 62.6), turned to 0 degrees
- moved U3 63.1 mm to (184.5, 72.5), turned to 0 degrees
- moved D52 54.3 mm to (237.3, 204.7)
- moved K52 54.3 mm to (238.8, 213.2)
- moved K51 54.3 mm to (187.7, 213.2)
- moved D51 54.3 mm to (189.2, 204.7)
- moved D11 54.3 mm to (321.2, 131.9)
- moved K21 54.3 mm to (288.5, 165.8)
- moved K48 54.3 mm to (351.4, 193.4)
- moved K12 54.3 mm to (341.4, 137.1)
- moved K34 54.3 mm to (310.5, 181.2)
- moved D46 54.3 mm to (312.3, 191.5)
- moved K47 54.3 mm to (332.6, 196.7)
- moved D31 54.3 mm to (252.8, 182.6)
- moved D43 54.3 mm to (256.1, 201.4)
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Connections:
- U2 pad 13: Col6 -> Col_
- U2 pad 2: Row4 -> Row1
- U2 pad 3: Row3 -> Row2
- U2 pad 4: Row2 -> Row3
- U2 pad 5: Row1 -> Row4
- U2 pad 6: Col1 -> Col6
- U3 pad 6: Col6 -> Col_
Routing:
- net Col1: track 52.6 -> 191.8 mm
- net Row4: track 213.9 -> 349.1 mm, vias 0 -> 1
- net Col12: track 52.6 -> 179.6 mm
- net Col2: track 52.6 -> 171.8 mm
- net Row3: track 213.9 -> 325.4 mm, vias 0 -> 1
- net Col11: track 52.6 -> 162.1 mm
- net Row1: track 213.9 -> 312.3 mm, vias 0 -> 1
- net Col3: track 52.6 -> 150.3 mm
- net Col6: track 75.5 -> 165.0 mm
- net Row2: track 213.9 -> 303.5 mm, vias 0 -> 1
- net Col10: track 52.6 -> 142.1 mm
- net Col4: track 52.6 -> 123.1 mm
- net Col7: track 73.7 -> 135.7 mm
- net Col5: track 52.6 -> 108.1 mm
- net Row5: track 90.7 -> 64.2 mm
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Other:
- board size 297.2 x 117 mm -> 298.3 x 117 mm

Commit message: Wire everything switch related
Parts:
- removed D49, D50, D51, D52, D53, D54: D, my_lib:D_SOD123_axial
- removed K49, K50, K51, K52, K53, K54: KEYSW, my_lib:MX-1U-Hotswap-Antishear
- K1, K10, K11, K12, K13, K14, K15, K16, K17, K18, K19, K2, K20, K21, K22, K23, K24, K25, K26, K27, K28, K29, K3, K30, K31, K32, K33, K34, K35, K36, K37, K38, K39, K4, K40, K41, K42, K43, K44, K45, K46, K47, K48, K5, K6, K7, K8, K9: footprint my_lib:MX-1U-Hotswap-Antishear -> my_lib:MX-1U-Hotswap-Antishear-flipped
- U1: value PIM447 -> Teensy3.2; footprint my_lib:PIM447 -> teensy:Teensy30_31_32_All_Pins
- U2: value Teensy3.2 -> ST7789_SPI; footprint teensy:Teensy30_31_32_All_Pins -> my_lib:ST7789_1.3_240x240
- U3: value ST7789_SPI -> PIM447; footprint my_lib:ST7789_1.3_240x240 -> my_lib:PIM447
- moved D12 332.1 mm to (45.7, -25.5), turned to 180 degrees
- moved D11 317.8 mm to (42.7, -21.2), turned to 180 degrees
- moved K12 313.7 mm to (38.1, 57.1), turned to 0 degrees
- moved D10 303.6 mm to (39.6, -16.9), turned to 180 degrees
- moved K11 302.4 mm to (38.1, 38.1), turned to 0 degrees
- moved D24 296.1 mm to (102.9, -25.5), turned to 180 degrees
- moved K10 293.6 mm to (38.1, 19.1), turned to 0 degrees
- moved D8 291.1 mm to (26.7, -25.5), turned to 180 degrees
- moved D9 289.6 mm to (36.6, -12.6), turned to 180 degrees
- moved K9 287.5 mm to (38.1, 0.00), turned to 0 degrees
- moved D23 282.9 mm to (99.8, -21.2), turned to 180 degrees
- moved D7 277.8 mm to (23.6, -21.2), turned to 180 degrees
- moved D22 269.9 mm to (96.8, -16.9), turned to 180 degrees
- moved K24 268.3 mm to (95.2, 57.1), turned to 0 degrees
- moved K8 264.3 mm to (19.1, 57.1), turned to 0 degrees
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Connections:
- D10 pad 1: Row1 -> Row2
- D11 pad 1: Row1 -> Row3
- D12 pad 1: Row1 -> Row4
- D13 pad 1: Row2 -> Row1
- D15 pad 1: Row2 -> Row3
- D16 pad 1: Row2 -> Row4
- D17 pad 1: Row2 -> Row1
- D19 pad 1: Row2 -> Row3
- D2 pad 1: Row1 -> Row2
- D20 pad 1: Row2 -> Row4
- D21 pad 1: Row2 -> Row1
- D23 pad 1: Row2 -> Row3
- D24 pad 1: Row2 -> Row4
- D25 pad 1: Row3 -> Row1
- D26 pad 1: Row3 -> Row2
- D28 pad 1: Row3 -> Row4
- D29 pad 1: Row3 -> Row1
- D3 pad 1: Row1 -> Row3
- D30 pad 1: Row3 -> Row2
- D32 pad 1: Row3 -> Row4
- D33 pad 1: Row3 -> Row1
- D34 pad 1: Row3 -> Row2
- D36 pad 1: Row3 -> Row4
- D37 pad 1: Row4 -> Row1
- D38 pad 1: Row4 -> Row2
- D39 pad 1: Row4 -> Row3
- D4 pad 1: Row1 -> Row4
- D41 pad 1: Row4 -> Row1
- D42 pad 1: Row4 -> Row2
- D43 pad 1: Row4 -> Row3
- D45 pad 1: Row4 -> Row1
- D46 pad 1: Row4 -> Row2
- D47 pad 1: Row4 -> Row3
- D6 pad 1: Row1 -> Row2
- D7 pad 1: Row1 -> Row3
- D8 pad 1: Row1 -> Row4
- K10 pad 1: Col10 -> Col3
- K11 pad 1: Col11 -> Col3
- K12 pad 1: Col12 -> Col3
- K13 pad 1: Col1 -> Col4
- K14 pad 1: Col2 -> Col4
- K15 pad 1: Col3 -> Col4
- K18 pad 1: Col6 -> Col5
- K19 pad 1: Col7 -> Col5
- K2 pad 1: Col2 -> Col1
- K20 pad 1: Col8 -> Col5
- K21 pad 1: Col9 -> Col6
- K22 pad 1: Col10 -> Col6
- K23 pad 1: Col11 -> Col6
- K24 pad 1: Col12 -> Col6
- K25 pad 1: Col1 -> Col7
- K26 pad 1: Col2 -> Col7
- K27 pad 1: Col3 -> Col7
- K28 pad 1: Col4 -> Col7
- K29 pad 1: Col5 -> Col8
- K3 pad 1: Col3 -> Col1
- K30 pad 1: Col6 -> Col8
- K31 pad 1: Col7 -> Col8
- K34 pad 1: Col10 -> Col9
- K35 pad 1: Col11 -> Col9
- K36 pad 1: Col12 -> Col9
- K37 pad 1: Col1 -> Col10
- K38 pad 1: Col2 -> Col10
- K39 pad 1: Col3 -> Col10
- K4 pad 1: Col4 -> Col1
- K40 pad 1: Col4 -> Col10
- K41 pad 1: Col5 -> Col11
- K42 pad 1: Col6 -> Col11
- K43 pad 1: Col7 -> Col11
- K44 pad 1: Col8 -> Col11
- K45 pad 1: Col9 -> Col12
- K46 pad 1: Col10 -> Col12
- K47 pad 1: Col11 -> Col12
- K5 pad 1: Col5 -> Col2
- K6 pad 1: Col6 -> Col2
- K7 pad 1: Col7 -> Col2
- K8 pad 1: Col8 -> Col2
- K9 pad 1: Col9 -> Col3
- U1 pad 1: VCC -> GND
- U1 pad 2: SDA -> Row4
- U1 pad 3: SCL -> Row3
- U1 pad 4: unconnected-(U1-Pad4) -> Row2
- U1 pad 5: GND -> Row1
- U2 pad 1: GND -> VCC
- U2 pad 10: Col5 -> unconnected-(U2-Pad10)
- U2 pad 2: Row1 -> unconnected-(U2-Pad2)
- U2 pad 3: Row2 -> GND
- U2 pad 4: Row3 -> Row5
- U2 pad 5: Row4 -> unconnected-(U2-Pad5)
- U2 pad 6: Col6 -> Col1
- U2 pad 7: Col2 -> LCD CS
- U2 pad 8: Col3 -> LCD RST
- U2 pad 9: Col4 -> LCD DC
- U3 pad 2: unconnected-(U3-Pad2) -> SDA
- U3 pad 3: GND -> SCL
- U3 pad 4: Row5 -> unconnected-(U3-Pad4)
- U3 pad 5: unconnected-(U3-Pad5) -> GND
Routing:
- net Row4: track 349.1 -> 235.1 mm, vias 1 -> 0
- net Row3: track 325.4 -> 241.5 mm, vias 1 -> 0
- net Col6: track 165.0 -> 88.3 mm
- net Net-(D48-Pad2): track 9.25 -> 82.6 mm
- net Net-(D32-Pad2): track 9.25 -> 82.6 mm
- net Net-(D36-Pad2): track 9.25 -> 82.6 mm
- net Net-(D44-Pad2): track 9.25 -> 82.6 mm
- net Net-(D40-Pad2): track 9.25 -> 82.6 mm
- net Net-(D28-Pad2): track 9.25 -> 82.6 mm
- net Net-(D16-Pad2): track 9.25 -> 79.1 mm
- net Net-(D12-Pad2): track 9.25 -> 79.1 mm
- net Net-(D24-Pad2): track 9.25 -> 79.1 mm
- net Net-(D4-Pad2): track 9.25 -> 79.1 mm
- net Net-(D8-Pad2): track 9.25 -> 79.1 mm
- net Net-(D20-Pad2): track 9.25 -> 79.1 mm
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Other:
- board size 298.3 x 117 mm -> 266.7 x 95.2 mm

Commit message: Cleanup
Parts:
- U1: footprint teensy:Teensy30_31_32_All_Pins -> my_lib:Teensy32
- moved D21 148.7 mm to (185.6, 104.3)
- moved D29 148.7 mm to (264.8, 104.3)
- moved D33 148.7 mm to (283.9, 104.3)
- moved D37 148.7 mm to (302.9, 104.3)
- moved D9 148.7 mm to (128.4, 104.3)
- moved K10 148.7 mm to (130.0, 135.9)
- moved K22 148.7 mm to (187.1, 135.9)
- moved K30 148.7 mm to (263.3, 135.9)
- moved K34 148.7 mm to (282.4, 135.9)
- moved K38 148.7 mm to (301.4, 135.9)
- moved D1 148.7 mm to (90.3, 104.3)
- moved D10 148.7 mm to (131.5, 100.0)
- moved D11 148.7 mm to (134.5, 95.7)
- moved D12 148.7 mm to (137.6, 91.3)
- moved D13 148.7 mm to (147.5, 104.3)
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Connections:
- U1 pad 29: Col11 -> (no net)
- U1 pad 30: Col12 -> (no net)
- U1 pad 31: unconnected-(U1-Pad31) -> (no net)
- U1 pad 32: unconnected-(U1-Pad32) -> (no net)
- U1 pad 33: VCC -> (no net)
Routing:
- net VCC: track 0.00 -> 78.9 mm
- net SCL: track 0.00 -> 63.6 mm
- net SDA: track 0.00 -> 58.8 mm
- net Col9: track 62.6 -> 107.2 mm
- net LCD DC: track 0.00 -> 23.4 mm
- net LCD RST: track 0.00 -> 23.0 mm
- net LCD CS: track 0.00 -> 19.1 mm
- net LCD LITE: track 0.00 -> 14.4 mm
- net Col1: track 176.9 -> 189.6 mm
- net Row5: track 0.00 -> 8.22 mm
- net Row2: track 250.0 -> 249.2 mm
- added copper zone on F.Cu, net GND
